File: pi-top_Glimmer.sch (KiCad schematic (older format))
At the start: 90 parts, among them J1 CONN_01X06, J2 CONN_02X03, Q1 IRFML8244, Q2 IRFML8244, Q3 IRFML8244, Q4 IRFML8244, Q5 IRFML8244, Q6 IRFML8244, Q7 IRFML8244, Q8 IRFML8244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

Commit message: Added solder jumper to IR Rcvr; README edits
Changed lines of the file:
@@
 LIBS:dmmt5401
 LIBS:7215
+LIBS:SolderJumpers
 LIBS:pi-top_Glimmer-cache
 EELAYER 26 0
@@
 $EndDescr
 $Sheet
-S 1000 6950 600  650
+S 1350 6750 600  650
 U 592048E0
 F0 "Sheet2" 60
@@
 	-1   0    0    -1
 $EndComp
-Text GLabel 1450 2800 2    39   Output ~ 0
+Text GLabel 1450 2800 2    39   UnSpc ~ 0
 AVR_RXI
-Text GLabel 1450 2900 2    39   Input ~ 0
+Text GLabel 1450 2900 2    39   UnSpc ~ 0
 AVR_TXO
 Text GLabel 1450 3000 2    39   UnSpc ~ 0
@@
 	6100 2000 6100 2500
 Connection ~ 6100 2350
-Text GLabel 5550 2600 2    39   Output ~ 0
+Text GLabel 5550 2600 2    39   UnSpc ~ 0
 AVR_TXO
-Text GLabel 5550 2500 2    39   Input ~ 0
+Text GLabel 5550 2500 2    39   UnSpc ~ 0
 AVR_RXI
 $Comp
